Commit message: made progress

File: src/murphy_description/urdf/murphy.urdf.xacro (robot description, xacro)
@@ -1,4 +1,29 @@
 <?xml version="1.0"?>
 <robot name="murphy" xmlns:xacro="http://www.ros.org/wiki/xacro">
+  <ros2_control name="MurphySystem" type="system">
+  <hardware>
+    <plugin>gz_ros2_control/GazeboSimSystem</plugin>
+  </hardware>
+  <joint name="front_left_wheel_joint">
+    <command_interface name="velocity"/>
+    <state_interface name="position"/>
+    <state_interface name="velocity"/>
+  </joint>
+  <joint name="rear_left_wheel_joint">
+    <command_interface name="velocity"/>
+    <state_interface name="position"/>
+    <state_interface name="velocity"/>
+  </joint>
+  <joint name="front_right_wheel_joint">
+    <command_interface name="velocity"/>
+    <state_interface name="position"/>
+    <state_interface name="velocity"/>
+  </joint>
+  <joint name="rear_right_wheel_joint">
+    <command_interface name="velocity"/>
+    <state_interface name="position"/>
+    <state_interface name="velocity"/>
+  </joint>
+</ros2_control>
   <xacro:property name="pi" value="3.14159265359"/>
   <xacro:property name="wheel_radius" value="0.07"/>
@@ -93,21 +118,4 @@
   <xacro:wheel name="rear_left_wheel"   x="-0.15" y="0.15"/>
   <xacro:wheel name="rear_right_wheel"  x="-0.15" y="-0.15"/>
-  <gazebo>
-  <plugin
-      filename="libgz-sim-diff-drive-system.so"
-      name="gz::sim::systems::DiffDrive">
-    <left_joint>front_left_wheel_joint</left_joint>
-    <left_joint>rear_left_wheel_joint</left_joint>
-    <right_joint>front_right_wheel_joint</right_joint>
-    <right_joint>rear_right_wheel_joint</right_joint>
-    <wheel_separation>0.3</wheel_separation>
-    <wheel_radius>${wheel_radius}</wheel_radius>
-    <topic>cmd_vel</topic>
-    <odom_topic>odom</odom_topic>
-    <tf_topic>tf</tf_topic>
-    <frame_id>odom</frame_id>
-    <child_frame_id>base_link</child_frame_id>
-  </plugin>
-</gazebo>
 <gazebo reference="lidar_link">
   <sensor name="lidar" type="gpu_lidar">
@@ -136,3 +144,9 @@
   </sensor>
 </gazebo>
+<gazebo>
+  <plugin filename="libgz_ros2_control-system.so"
+          name="gz_ros2_control::GazeboSimROS2ControlPlugin">
+    <parameters>$(find murphy_description)/config/controllers.yaml</parameters>
+  </plugin>
+</gazebo>
 </robot>
